File: Jove.kicad_sch (KiCad schematic)
At the start: 155 parts, among them J1 Resonance CV, J2 Bipolar Freq CV, J3 Unipolar Freq CV, J4 Input2, J5 Input2, J6 out, J7 prog, P1 CONN_02X05, Q1 BCM857BS, Q2 BCM857BS, Q3 J112, Q4 J112, Q5 J112, Q6 J112, SW1 SW_Push_DPDT, U1 TL072-, U10 STC8, U106 L78L05, U12 TL072-, U2 TL072-, U3 TL072-, U4 TL072-, U5 LM13700, U6 LM13700, U7 LM13700, U8 DG409

Commit message: add batch 2 changes
Parts:
- C1, C11, C28, C29: LCSC Part # (none) -> C1653
- C10, C23, C24: LCSC Part # (none) -> C7171
- C18, C25, C6, C7: LCSC Part # (none) -> C1664
- C2, C5: LCSC Part # (none) -> C1671
- C3, C8: LCSC Part # (none) -> C1669
- C4, C9: LCSC Part # (none) -> C1663
- D10, D5, D6: value 1N914 -> 1N4148WS; LCSC Part # (none) -> C2128
- D3: LCSC Part # (none) -> C2286
- D8, D9: LCSC Part # (none) -> C7420331
- P1: LCSC Part # (none) -> C5383106
- Q1, Q2: LCSC Part # (none) -> C105887
- Q3, Q4, Q5, Q6: LCSC Part # (none) -> C258195
- R1, R19, R49, R70, R71: LCSC Part # (none) -> C25804
- R10: LCSC Part # (none) -> C25822
- R11, R21, R28: LCSC Part # (none) -> C22935
- R12, R54: value 1K -> 1k; LCSC Part # (none) -> C21190
- R13, R14, R18, R50: LCSC Part # (none) -> C25819
- R15: LCSC Part # (none) -> C22807
- R16: LCSC Part # (none) -> C23162
- R17: LCSC Part # (none) -> C23189
- R2, R24, R26, R3, R4, R44, R45, R47, R48, R7, R73, R74, R75, R76, R77, R78, R8: value 100K -> 100k; LCSC Part # (none) -> C25803
- R20, R27: LCSC Part # (none) -> C22843
- R22: LCSC Part # (none) -> C25981
- R23: LCSC Part # (none) -> C4177
- R25: LCSC Part # (none) -> C23253
- R29, R35, R37, R52, R60, R63: LCSC Part # (none) -> C23231
- R30, R36, R38, R53, R62, R65: LCSC Part # (none) -> C23204
- R31, R32, R39, R55, R56, R68: LCSC Part # (none) -> C25810
- R33, R34, R40, R46, R57, R69: LCSC Part # (none) -> C4216
- R41: LCSC Part # (none) -> C25803
- R42, R43: LCSC Part # (none) -> C23206
- R5, R6: LCSC Part # (none) -> C25811
- R51: LCSC Part # (none) -> C23137
- R58: LCSC Part # (none) -> C21190
- R59, R61: LCSC Part # (none) -> C23138
- R64: value 330 -> 1k; LCSC Part # (none) -> C21190
- R66, R67: value 10 -> PPTC; LCSC Part # (none) -> C2649905
- R72: LCSC Part # (none) -> C22965
- R79, R80: LCSC Part # (none) -> C23178
- R9: LCSC Part # (none) -> C25805
- U1, U12, U2, U3, U4: value TL072- -> TL072; LCSC Part # (none) -> C6961
- U10: value STC8 -> STC8G1K08-36I; LCSC Part # (none) -> C713818
- U5, U6, U7: LCSC Part # (none) -> C521166
- U8: LCSC Part # (none) -> C142533
- VR1, VR2, VR3, VR4, VR6: value 50K -> 100k
- VR5, VR7: LCSC Part # (none) -> C128545
Other:
- note removed: "REPLACE WITH PTC FUSE IN NEXT REVISION"
